File: ads1293_board/iter2/pcb_itr2.kicad_sch (KiCad schematic)
At the start: 23 parts, among them J1 Conn_01x05_Pin, J2 RSTB_J, J3 Breakout Pins, U1 ADS1293CISQ/NOPB, U2 SPX5205M5-L-5-0/TR, Y1 4.096 MHz

Commit message: adding gerber files
Parts:
- added D1: LED, LED_SMD:LED_0603_1608Metric, symbol Device:LED
- added J4: Power Input, Connector_PinHeader_1.00mm:PinHeader_1x02_P1.00mm_Vertical, symbol Connector:Conn_01x02_Pin
- added R10: 22K Ohm, Resistor_SMD:R_0603_1608Metric, symbol Device:R_Small
- added R11: 12K Ohm, Resistor_SMD:R_0603_1608Metric, symbol Device:R_Small
- added R12: 220 Ohms, Resistor_SMD:R_0603_1608Metric, symbol Device:R_Small
Connections:
- net +3.3V: now also C3.2, C8.1, U1.28 (VDD), U1.29 (EPAD), U2.5 (OUT), R11.2, R12.1
- net GND: now also D1.1 (K), J4.2 (Pin_2), R10.1
- net at U2.4 (RST/ADJ): now also R10.2, R11.1
- net +9V renamed +5V
- net +5V: now also J4.1 (Pin_1)
- new net: D1.2 (A), R12.2
- no-connect marks 5 -> 4
Other:
- note added: "Crystal"
- moved on the sheet: C8, U2
