File: ads1293_board/iter2/pcb_itr2.kicad_sch (KiCad schematic)
At the start: 28 parts, among them J1 Conn_01x05_Pin, J2 RSTB_J, J3 Breakout Pins, J4 Power Input, U1 ADS1293CISQ/NOPB, U2 SPX5205M5-L-5-0/TR, Y1 4.096 MHz

Commit message: uploaded files for manufacturing
Parts:
- J1: footprint Connector_PinHeader_1.00mm:PinHeader_1x05_P1.00mm_Vertical -> Connector_PinHeader_2.54mm:PinHeader_1x05_P2.54mm_Vertical
- J3: footprint Connector_PinHeader_1.00mm:PinHeader_1x06_P1.00mm_Vertical -> Connector_PinHeader_2.54mm:PinHeader_1x06_P2.54mm_Vertical
- J4: footprint Connector_PinHeader_1.00mm:PinHeader_1x02_P1.00mm_Vertical -> Connector_PinHeader_2.54mm:PinHeader_1x02_P2.54mm_Vertical
Changed lines of the file:
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@@
 			)
 		)
-		(property "Footprint" "Connector_PinHeader_1.00mm:PinHeader_1x06_P1.00mm_Vertical"
+		(property "Footprint" "Connector_PinHeader_2.54mm:PinHeader_1x06_P2.54mm_Vertical"
 			(at 187.96 86.36 0)
 			(effects
@@
 			)
 		)
-		(property "Footprint" "Connector_PinHeader_1.00mm:PinHeader_1x02_P1.00mm_Vertical"
+		(property "Footprint" "Connector_PinHeader_2.54mm:PinHeader_1x02_P2.54mm_Vertical"
 			(at 124.46 132.08 0)
 			(effects
@@
 			)
 		)
-		(property "Footprint" "Connector_PinHeader_1.00mm:PinHeader_1x05_P1.00mm_Vertical"
+		(property "Footprint" "Connector_PinHeader_2.54mm:PinHeader_1x05_P2.54mm_Vertical"
 			(at 76.2 60.96 0)
 			(effects

Commit message: more docs
Parts:
- R10: value 22K Ohm -> 12K Ohm
- R11: value 12K Ohm -> 22K Ohm
Changed lines of the file:
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@@
 		(fields_autoplaced yes)
 		(property "Reference" "R11"
-			(at 182.88 128.27 0)
+			(at 182.88 128.2699 0)
 			(effects
 				(font
@@
 			)
 		)
-		(property "Value" "12K Ohm"
-			(at 182.88 130.81 0)
+		(property "Value" "22K Ohm"
+			(at 182.88 130.8099 0)
 			(effects
 				(font
@@
 		(fields_autoplaced yes)
 		(property "Reference" "R10"
-			(at 182.88 115.57 0)
+			(at 182.88 115.5699 0)
 			(effects
 				(font
@@
 			)
 		)
-		(property "Value" "22K Ohm"
-			(at 182.88 118.11 0)
-			(effects
-				(font
+		(property "Value" "12K Ohm"
+			(at 182.88 118.1099 0)
+			(effects
+				(font
