File: ads1293_board/iter2/pcb_itr2.kicad_pcb (KiCad board)
At the start: 2 copper layers, 23.1 x 25.6 mm, 23 parts, among them J1 Conn_01x05_Pin, J2 RSTB_J, J3 Breakout Pins, U1 ADS1293CISQ/NOPB, U2 SPX5205M5-L-5-0/TR, Y1 4.096 MHz

Commit message: adding gerber files
Parts:
- added D1: LED, LED_SMD:LED_0603_1608Metric, F.Cu at (122.3, 69.2)
- added J4: Power Input, Connector_PinHeader_1.00mm:PinHeader_1x02_P1.00mm_Vertical, F.Cu at (125.2, 71.4)
- added R10: 22K Ohm, Resistor_SMD:R_0603_1608Metric, F.Cu at (119.2, 69.2)
- added R11: 12K Ohm, Resistor_SMD:R_0603_1608Metric, F.Cu at (119.2, 67.4)
- added R12: 220 Ohms, Resistor_SMD:R_0603_1608Metric, F.Cu at (122.3, 67.4)
- moved Y1 2.63 mm to (130.2, 69.1)
Connections:
- net +9V renamed +5V
- C3 pad 2: Net-(U1-VDD) -> +3.3V
- C8 pad 1: Net-(U1-VDD) -> +3.3V
- U1 pad 28: Net-(U1-VDD) -> +3.3V
- U1 pad 29: unconnected-(U1-EPAD-Pad29) -> +3.3V
- U2 pad 4: unconnected-(U2-RST/ADJ-Pad4) -> Net-(U2-RST/ADJ)
- U2 pad 5: Net-(U1-VDD) -> +3.3V
Routing:
- net +3.3V: track 18.0 -> 48.9 mm
- net Net-(U1-VDD): track 11.0 -> 0.00 mm
- net Net-(U2-RST/ADJ): track 0.00 -> 8.86 mm
- net GND: track 34.6 -> 42.5 mm
- net +5V: track 3.62 -> 8.99 mm, vias 0 -> 2
- net Net-(D1-A): track 0.00 -> 1.81 mm
- net XTAL1: track 10.8 -> 12.1 mm
- net XTAL2: track 14.6 -> 13.5 mm, vias 2 -> 4
Other:
- board size 23.1 x 25.6 mm -> 23.5 x 25.6 mm
- board text added: "+"
- board text added: "-"
