File: ads1293_board/iter2/pcb_itr2.kicad_pcb (KiCad board)
At the start: 2 copper layers, 23.5 x 25.6 mm, 28 parts, among them J1 Conn_01x05_Pin, J2 RSTB_J, J3 Breakout Pins, J4 Power Input, U1 ADS1293CISQ/NOPB, U2 SPX5205M5-L-5-0/TR, Y1 4.096 MHz

Commit message: uploaded files for manufacturing
Parts:
- J1: footprint Connector_PinHeader_1.00mm:PinHeader_1x05_P1.00mm_Vertical -> Connector_PinHeader_2.54mm:PinHeader_1x05_P2.54mm_Vertical
- J3: footprint Connector_PinHeader_1.00mm:PinHeader_1x06_P1.00mm_Vertical -> Connector_PinHeader_2.54mm:PinHeader_1x06_P2.54mm_Vertical
- J4: footprint Connector_PinHeader_1.00mm:PinHeader_1x02_P1.00mm_Vertical -> Connector_PinHeader_2.54mm:PinHeader_1x02_P2.54mm_Vertical
- moved J3 6.02 mm to (137.5, 90.7)
- moved R4 5.15 mm to (137.5, 73.0)
- moved J1 1.26 mm to (119.5, 78.0)
- moved J2 0.74 mm to (137.5, 75.0)
Routing:
- net Net-(J3-Pin_1): track 3.15 -> 10.1 mm
- net Net-(U1-RSTB): track 6.31 -> 12.4 mm
- net Net-(J3-Pin_2): track 2.95 -> 7.87 mm
- net Net-(J3-Pin_3): track 2.74 -> 6.05 mm
- net Net-(J3-Pin_6): track 2.98 -> 6.14 mm
- net Net-(J3-Pin_4): track 2.57 -> 5.26 mm
- net Net-(J3-Pin_5): track 2.77 -> 5.30 mm
- net Net-(J1-Pin_5): track 4.76 -> 6.55 mm
Other:
- board size 23.5 x 25.6 mm -> 23.5 x 28.1 mm

Commit message: more docs
Parts:
- R10: value 22K Ohm -> 12K Ohm
- R11: value 12K Ohm -> 22K Ohm
Changed lines of the file:
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@@
 			)
 		)
-		(property "Value" "12K Ohm"
+		(property "Value" "22K Ohm"
 			(at 0 1.43 0)
 			(layer "F.Fab")
@@
 			)
 		)
-		(property "Value" "22K Ohm"
+		(property "Value" "12K Ohm"
 			(at 0 1.43 0)
 			(layer "F.Fab")
@@
 	)
 	(segment
-		(start 124.2875 70.4)
-		(end 123.0875 69.2)
-		(width 0.25)
-		(layer "F.Cu")
-		(net 5)
-	)
-	(segment
 		(start 129.23666 78.93196)
 		(end 129.23666 79.737646)
@@
 	)
 	(segment
+		(start 125.2 68.86)
+		(end 123.4275 68.86)
+		(width 0.25)
+		(layer "F.Cu")
+		(net 5)
+	)
+	(segment
+		(start 123.4275 68.86)
+		(end 123.0875 69.2)
+		(width 0.25)
+		(layer "F.Cu")
+		(net 5)
+	)
+	(segment
 		(start 120.088899 71.4)
 		(end 121.425 71.4)
@@
 	)
 	(segment
+		(start 125.2 68.86)
+		(end 125.86 68.86)
+		(width 0.25)
+		(layer "F.Cu")
+		(net 5)
+	)
+	(segment
 		(start 132.652395 86.113381)
 		(end 131.73666 85.197646)
@@
 		(net 5)
 	)
-	(segment
-		(start 125.2 70.4)
-		(end 124.2875 70.4)
-		(width 0.25)
-		(layer "F.Cu")
-		(net 5)
-	)
 	(via
 		(at 132.900925 86.113381)
@@
 	)
 	(segment
-		(start 118.35 69.175)
-		(end 118.375 69.2)
+		(start 117.382098 71.092902)
+		(end 117.382098 74.2571)
 		(width 0.25)
 		(layer "F.Cu")
@@
 	)
 	(segment
-		(start 117.382098 71.092902)
-		(end 117.382098 74.2571)
+		(start 118.35 67.4)
+		(end 118.35 69.175)
 		(width 0.25)
 		(layer "F.Cu")
@@
 	)
 	(segment
-		(start 118.35 67.4)
-		(end 118.35 69.175)
+		(start 118.35 69.175)
+		(end 118.375 69.2)
 		(width 0.25)
 		(layer "F.Cu")
